Commit message: replace rotor_description with quad_description

File: quad_description/urdf/component_snippets.xacro (robot description, xacro)
@@ -344,5 +344,5 @@
         <origin xyz="0 0 0" rpy="0 0 0" />
         <geometry>
-          <mesh filename="package://rotors_description/meshes/vi_sensor.dae" scale="1 1 1" />
+          <mesh filename="package://quad_description/meshes/vi_sensor.dae" scale="1 1 1" />
         </geometry>
       </visual>

File: quad_description/urdf/iris.xacro (robot description, xacro)
@@ -41,5 +41,5 @@
   </xacro:property>
   <!-- Included URDF Files -->
-  <xacro:include filename="$(find rotors_description)/urdf/multirotor_base.xacro" />
+  <xacro:include filename="$(find quad_description)/urdf/multirotor_base.xacro" />
   <!-- Instantiate multirotor_base_macro once -->
   <xacro:multirotor_base_macro

File: quad_description/urdf/iris_base.xacro (robot description, xacro)
@@ -1,7 +1,7 @@
 <?xml version="1.0"?>
 <robot name="iris" xmlns:xacro="http://ros.org/wiki/xacro">
-  <xacro:include filename="$(find rotors_description)/urdf/component_snippets.xacro" />
+  <xacro:include filename="$(find quad_description)/urdf/component_snippets.xacro" />
   <!-- Instantiate iris "mechanics" -->
-  <xacro:include filename="$(find rotors_description)/urdf/iris.xacro" />
+  <xacro:include filename="$(find quad_description)/urdf/iris.xacro" />
   <!-- Instantiate a controller. -->
   <xacro:controller_plugin_macro

File: quad_description/urdf/kit_c.urdf (robot description, URDF)
Before this commit: robot quad, 6 links, 5 joints
Links:
- link base_link_inertia: geometry collision box size=0.3 0.3 0.17; visual mesh filename=package://quad_description/meshes/hummingbird.dae scale=1 1 1
- link rotor_0: geometry collision cylinder length=0.005 radius=0.14; visual mesh filename=package://quad_description/meshes/propeller_ccw.dae scale=.12 .12 .12
- link rotor_1: geometry collision cylinder length=0.005 radius=0.14; visual mesh filename=package://quad_description/meshes/propeller_cw.dae scale=.12 .12 .12
- link rotor_2: geometry collision cylinder length=0.005 radius=0.14; visual mesh filename=package://quad_description/meshes/propeller_ccw.dae scale=.12 .12 .12
- link rotor_3: geometry collision cylinder length=0.005 radius=0.14; visual mesh filename=package://quad_description/meshes/propeller_cw.dae scale=.12 .12 .12

File: quad_description/urdf/multirotor_base.xacro (robot description, xacro)
@@ -35,5 +35,5 @@
         <origin xyz="0 0 0" rpy="0 0 0" />
         <geometry>
-          <mesh filename="package://rotors_description/meshes/${mesh_file}"
+          <mesh filename="package://quad_description/meshes/${mesh_file}"
             scale="${mesh_scale}" />
           <!-- <box size="${body_width} ${body_width} ${body_height}"/> --> <!-- [m] [m] [m] -->
@@ -81,6 +81,6 @@
         <geometry>
           <!-- <cylinder length="0.005" radius="${radius_rotor}"/> --> <!-- [m] -->
-          <!-- <mesh filename="package://rotors_description/meshes/propeller_${direction}.dae" -->
-          <mesh filename="package://rotors_description/meshes/${mesh}_${direction}.dae"
+          <!-- <mesh filename="package://quad_description/meshes/propeller_${direction}.dae" -->
+          <mesh filename="package://quad_description/meshes/${mesh}_${direction}.dae"
             scale="${mesh_scale}" />
           <!-- <box size="${2*radius_rotor} 0.01 0.005"/> -->

File: quad_description/urdf/sensors/sonar_sensor.urdf.xacro (robot description, xacro)
@@ -17,5 +17,5 @@
         <geometry>
           <!--<box size="0.01 0.01 0.01" /> -->
-          <mesh filename="package://rotors_description/meshes/max_sonar_ez4.dae"/>
+          <mesh filename="package://quad_description/meshes/max_sonar_ez4.dae"/>
         </geometry>
       </visual>

File: quad_description/urdf/sensors/static_camera.gazebo.xacro (robot description, xacro)
@@ -5,5 +5,5 @@
   <xacro:property name="bag_file" value="static_camera.bag" />
   <!-- Instantiate static_camera "mechanics" -->
-  <xacro:include filename="$(find rotors_description)/urdf/static_camera.urdf.xacro" />
+  <xacro:include filename="$(find quad_description)/urdf/static_camera.urdf.xacro" />
 <gazebo>
     <static>true</static>
